Commit message: fix: tf publishing bridge

File: src/gazebo_sim/robots/fishbot_v2_3d/urdf/fishbot_v2_3d.xacro (robot description, xacro)
@@ -34,4 +34,5 @@
   <xacro:property name="imu_topic" value="${topic_prefix + '/' + imu_pub if topic_prefix else '/' + imu_pub}"/>
   <xacro:property name="cmd_vel_topic" value="${topic_prefix + '/cmd_vel' if topic_prefix else '/cmd_vel'}"/>
+  <xacro:property name="tf_topic" value="/tf"/>
   <xacro:property name="wheel_radius" value="${wheel_geom['radius']}"/>
   <xacro:property name="wheel_length" value="${wheel_geom['length']}"/>
@@ -216,4 +217,5 @@
       <topic>${cmd_vel_topic}</topic>
       <odom_topic>${odom_topic}</odom_topic>
+      <tf_topic>${tf_topic}</tf_topic>
       <frame_id>${odom_frame_prefixed}</frame_id>
       <child_frame_id>${base_frame_prefixed}</child_frame_id>

Commit message: feat: add the second third-wheel

File: src/gazebo_sim/robots/fishbot_v2_3d/urdf/fishbot_v2_3d.xacro (robot description, xacro)
@@ -213,4 +213,30 @@
     <axis xyz="0 1 0"/>
   </joint>
+  <!-- Second caster for stability -->
+  <link name="caster2_link">
+    <visual>
+      <origin xyz="0 0 0" rpy="1.57079 0 0"/>
+      <geometry>
+        <sphere radius="${caster_radius}"/>
+      </geometry>
+    </visual>
+    <collision>
+      <origin xyz="0 0 0" rpy="1.57079 0 0"/>
+      <geometry>
+        <sphere radius="${caster_radius}"/>
+      </geometry>
+    </collision>
+    <inertial>
+      <mass value="${caster_mass}"/>
+      <inertia ixx="${wheel_inertia}" ixy="0" ixz="0" iyy="${wheel_inertia}" iyz="0" izz="${wheel_inertia}"/>
+    </inertial>
+  </link>
+  <!-- Second caster center at caster_radius -> bottom at z = 0 -->
+  <joint name="caster2_joint" type="fixed">
+    <parent link="${base_frame}"/>
+    <child link="caster2_link"/>
+    <origin xyz="-0.06 0.0 ${caster_radius}" rpy="0 0 0"/>
+    <axis xyz="0 1 0"/>
+  </joint>
   <!-- ========================================================= -->
   <!-- GAZEBO PLUGINS / EXTRAS                                   -->
@@ -223,4 +249,17 @@
     <mu1 value="0.0"/>
     <mu2 value="0.0"/>
+    <slip1 value="1.0"/>
+    <slip2 value="1.0"/>
+    <kp value="1000000.0"/>
+    <kd value="10.0"/>
+  </gazebo>
+  <gazebo reference="caster2_link">
+    <material>Gazebo/Black</material>
+  </gazebo>
+  <gazebo reference="caster2_link">
+    <mu1 value="0.0"/>
+    <mu2 value="0.0"/>
+    <slip1 value="1.0"/>
+    <slip2 value="1.0"/>
     <kp value="1000000.0"/>
     <kd value="10.0"/>
@@ -257,4 +296,7 @@
   </gazebo>
   <gazebo reference="caster_link">
+    <visual><laser_retro>${laser_retro}</laser_retro></visual>
+  </gazebo>
+  <gazebo reference="caster2_link">
     <visual><laser_retro>${laser_retro}</laser_retro></visual>
   </gazebo>
