Commit message: feat: put the robot frames into robot namespace

File: src/gazebo_sim/robots/fishbot_mid360/urdf/fishbot_mid360.xacro (robot description, xacro)
@@ -2,5 +2,8 @@
 <robot xmlns:xacro="http://www.ros.org/wiki/xacro" name="fishbot_mid360">
   <xacro:arg name="config_file" default="$(find gazebo_sim)/robots/fishbot_mid360/config/fishbot_mid360.yaml"/>
+  <xacro:arg name="robot_namespace" default=""/>
   <xacro:property name="config_file" value="$(arg config_file)"/>
+  <xacro:property name="robot_namespace" value="$(arg robot_namespace)"/>
+  <xacro:property name="frame_prefix" value="${robot_namespace + '/' if robot_namespace != '' else ''}"/>
   <xacro:property name="cfg" value="${xacro.load_yaml(config_file)}"/>
   <xacro:property name="robot_cfg" value="${cfg['robot']}"/>
@@ -17,4 +20,9 @@
   <xacro:property name="lidar_frame" value="${robot_cfg['lidar_frame']}"/>
   <xacro:property name="imu_frame" value="${robot_cfg['imu_frame']}"/>
+  <xacro:property name="odom_frame" value="${robot_cfg['odom_frame']}"/>
+  <xacro:property name="base_frame_prefixed" value="${frame_prefix + base_frame}"/>
+  <xacro:property name="lidar_frame_prefixed" value="${frame_prefix + lidar_frame}"/>
+  <xacro:property name="imu_frame_prefixed" value="${frame_prefix + imu_frame}"/>
+  <xacro:property name="odom_frame_prefixed" value="${frame_prefix + odom_frame}"/>
   <xacro:property name="odom_pub" value="${robot_cfg['odom_pub']}"/>
   <xacro:property name="lidar_pub" value="${robot_cfg['lidar_pub']}"/>
@@ -194,5 +202,5 @@
     <plugin name="diff_drive" filename="libgazebo_ros_diff_drive.so">
       <ros>
-        <remapping>cmd_vel:=cmd_vel</remapping>
+        <namespace>${robot_namespace}</namespace>
         <remapping>odom:=${odom_pub}</remapping>
       </ros>
@@ -206,7 +214,6 @@
       <publish_odom>${'true' if diff_drive_cfg['publish_odom'] else 'false'}</publish_odom>
       <publish_odom_tf>${'true' if diff_drive_cfg['publish_odom_tf'] else 'false'}</publish_odom_tf>
-      <publish_wheel_tf>${'true' if diff_drive_cfg['publish_wheel_tf'] else 'false'}</publish_wheel_tf>
-      <odometry_frame>odom</odometry_frame>
-      <robot_base_frame>${base_frame}</robot_base_frame>
+      <odometry_frame>${odom_frame_prefixed}</odometry_frame>
+      <robot_base_frame>${base_frame_prefixed}</robot_base_frame>
     </plugin>
   </gazebo>
@@ -215,4 +222,5 @@
       <plugin filename="libgazebo_ros_imu_sensor.so" name="imu_plugin">
         <ros>
+          <namespace>${robot_namespace}</namespace>
           <remapping>~/out:=${imu_pub}</remapping>
         </ros>
@@ -312,8 +320,9 @@
       <plugin name="lidar_plugin" filename="libgazebo_ros_ray_sensor.so">
         <ros>
+          <namespace>${robot_namespace}</namespace>
           <remapping>~/out:=${lidar_pub}</remapping>
         </ros>
         <output_type>sensor_msgs/PointCloud2</output_type>
-        <frame_name>${lidar_frame}</frame_name>
+        <frame_name>${lidar_frame_prefixed}</frame_name>
       </plugin>
     </sensor>

File: src/gazebo_sim/robots/fishbot_v1/urdf/fishbot_v1.xacro (robot description, xacro)
@@ -2,5 +2,8 @@
 <robot xmlns:xacro="http://www.ros.org/wiki/xacro" name="fishbot_v1">
   <xacro:arg name="config_file" default="$(find gazebo_sim)/robots/fishbot_v1/config/fishbot_v1.yaml"/>
+  <xacro:arg name="robot_namespace" default=""/>
   <xacro:property name="config_file" value="$(arg config_file)"/>
+  <xacro:property name="robot_namespace" value="$(arg robot_namespace)"/>
+  <xacro:property name="frame_prefix" value="${robot_namespace + '/' if robot_namespace != '' else ''}"/>
   <xacro:property name="cfg" value="${xacro.load_yaml(config_file)}"/>
   <xacro:property name="robot_cfg" value="${cfg['robot']}"/>
@@ -17,4 +20,9 @@
   <xacro:property name="lidar_frame" value="${robot_cfg['lidar_frame']}"/>
   <xacro:property name="imu_frame" value="${robot_cfg['imu_frame']}"/>
+  <xacro:property name="odom_frame" value="${robot_cfg['odom_frame']}"/>
+  <xacro:property name="base_frame_prefixed" value="${frame_prefix + base_frame}"/>
+  <xacro:property name="lidar_frame_prefixed" value="${frame_prefix + lidar_frame}"/>
+  <xacro:property name="imu_frame_prefixed" value="${frame_prefix + imu_frame}"/>
+  <xacro:property name="odom_frame_prefixed" value="${frame_prefix + odom_frame}"/>
   <xacro:property name="odom_pub" value="${robot_cfg['odom_pub']}"/>
   <xacro:property name="lidar_pub" value="${robot_cfg['lidar_pub']}"/>
@@ -194,5 +202,5 @@
     <plugin name="diff_drive" filename="libgazebo_ros_diff_drive.so">
       <ros>
-        <remapping>cmd_vel:=cmd_vel</remapping>
+        <namespace>${robot_namespace}</namespace>
         <remapping>odom:=${odom_pub}</remapping>
       </ros>
@@ -206,7 +214,6 @@
       <publish_odom>${'true' if diff_drive_cfg['publish_odom'] else 'false'}</publish_odom>
       <publish_odom_tf>${'true' if diff_drive_cfg['publish_odom_tf'] else 'false'}</publish_odom_tf>
-      <publish_wheel_tf>${'true' if diff_drive_cfg['publish_wheel_tf'] else 'false'}</publish_wheel_tf>
-      <odometry_frame>odom</odometry_frame>
-      <robot_base_frame>${base_frame}</robot_base_frame>
+      <odometry_frame>${odom_frame_prefixed}</odometry_frame>
+      <robot_base_frame>${base_frame_prefixed}</robot_base_frame>
     </plugin>
   </gazebo>
@@ -215,4 +222,5 @@
       <plugin filename="libgazebo_ros_imu_sensor.so" name="imu_plugin">
         <ros>
+          <namespace>${robot_namespace}</namespace>
           <remapping>~/out:=${imu_pub}</remapping>
         </ros>
@@ -306,8 +314,9 @@
       <plugin name="lidar_plugin" filename="libgazebo_ros_ray_sensor.so">
         <ros>
+          <namespace>${robot_namespace}</namespace>
           <remapping>~/out:=${lidar_pub}</remapping>
         </ros>
         <output_type>sensor_msgs/PointCloud2</output_type>
-        <frame_name>${lidar_frame}</frame_name>
+        <frame_name>${lidar_frame_prefixed}</frame_name>
       </plugin>
     </sensor>

File: src/gazebo_sim/robots/fishbot_v2_3d/urdf/fishbot_v2_3d.xacro (robot description, xacro)
@@ -2,5 +2,8 @@
 <robot xmlns:xacro="http://www.ros.org/wiki/xacro" name="fishbot_v2_3d">
   <xacro:arg name="config_file" default="$(find gazebo_sim)/robots/fishbot_v2_3d/config/fishbot_v2_3d.yaml"/>
+  <xacro:arg name="robot_namespace" default=""/>
   <xacro:property name="config_file" value="$(arg config_file)"/>
+  <xacro:property name="robot_namespace" value="$(arg robot_namespace)"/>
+  <xacro:property name="frame_prefix" value="${robot_namespace + '/' if robot_namespace != '' else ''}"/>
   <xacro:property name="cfg" value="${xacro.load_yaml(config_file)}"/>
   <xacro:property name="robot_cfg" value="${cfg['robot']}"/>
@@ -17,4 +20,9 @@
   <xacro:property name="lidar_frame" value="${robot_cfg['lidar_frame']}"/>
   <xacro:property name="imu_frame" value="${robot_cfg['imu_frame']}"/>
+  <xacro:property name="odom_frame" value="${robot_cfg['odom_frame']}"/>
+  <xacro:property name="base_frame_prefixed" value="${frame_prefix + base_frame}"/>
+  <xacro:property name="lidar_frame_prefixed" value="${frame_prefix + lidar_frame}"/>
+  <xacro:property name="imu_frame_prefixed" value="${frame_prefix + imu_frame}"/>
+  <xacro:property name="odom_frame_prefixed" value="${frame_prefix + odom_frame}"/>
   <xacro:property name="odom_pub" value="${robot_cfg['odom_pub']}"/>
   <xacro:property name="lidar_pub" value="${robot_cfg['lidar_pub']}"/>
@@ -194,5 +202,5 @@
     <plugin name="diff_drive" filename="libgazebo_ros_diff_drive.so">
       <ros>
-        <remapping>cmd_vel:=cmd_vel</remapping>
+        <namespace>${robot_namespace}</namespace>
         <remapping>odom:=${odom_pub}</remapping>
       </ros>
@@ -206,7 +214,6 @@
       <publish_odom>${'true' if diff_drive_cfg['publish_odom'] else 'false'}</publish_odom>
       <publish_odom_tf>${'true' if diff_drive_cfg['publish_odom_tf'] else 'false'}</publish_odom_tf>
-      <publish_wheel_tf>${'true' if diff_drive_cfg['publish_wheel_tf'] else 'false'}</publish_wheel_tf>
-      <odometry_frame>odom</odometry_frame>
-      <robot_base_frame>${base_frame}</robot_base_frame>
+      <odometry_frame>${odom_frame_prefixed}</odometry_frame>
+      <robot_base_frame>${base_frame_prefixed}</robot_base_frame>
     </plugin>
   </gazebo>
@@ -215,4 +222,5 @@
       <plugin filename="libgazebo_ros_imu_sensor.so" name="imu_plugin">
         <ros>
+          <namespace>${robot_namespace}</namespace>
           <remapping>~/out:=${imu_pub}</remapping>
         </ros>
@@ -312,8 +320,9 @@
       <plugin name="lidar_plugin" filename="libgazebo_ros_ray_sensor.so">
         <ros>
+          <namespace>${robot_namespace}</namespace>
           <remapping>~/out:=${lidar_pub}</remapping>
         </ros>
         <output_type>sensor_msgs/PointCloud2</output_type>
-        <frame_name>${lidar_frame}</frame_name>
+        <frame_name>${lidar_frame_prefixed}</frame_name>
       </plugin>
     </sensor>

Commit message: feat: increase the reflectivity of the robots

File: src/gazebo_sim/robots/fishbot_mid360/urdf/fishbot_mid360.xacro (robot description, xacro)
@@ -21,4 +21,5 @@
   <xacro:property name="imu_frame" value="${robot_cfg['imu_frame']}"/>
   <xacro:property name="odom_frame" value="${robot_cfg['odom_frame']}"/>
+  <xacro:property name="laser_retro" value="${robot_cfg.get('laser_retro', 0.0)}"/>
   <xacro:property name="base_frame_prefixed" value="${frame_prefix + base_frame}"/>
   <xacro:property name="lidar_frame_prefixed" value="${frame_prefix + lidar_frame}"/>
@@ -214,7 +215,20 @@
       <publish_odom>${'true' if diff_drive_cfg['publish_odom'] else 'false'}</publish_odom>
       <publish_odom_tf>${'true' if diff_drive_cfg['publish_odom_tf'] else 'false'}</publish_odom_tf>
+      <tf_prefix>${frame_prefix}</tf_prefix>
       <odometry_frame>${odom_frame_prefixed}</odometry_frame>
       <robot_base_frame>${base_frame_prefixed}</robot_base_frame>
     </plugin>
+  </gazebo>
+  <gazebo reference="${base_frame}">
+    <laserRetro>${laser_retro}</laserRetro>
+  </gazebo>
+  <gazebo reference="left_wheel_link">
+    <laserRetro>${laser_retro}</laserRetro>
+  </gazebo>
+  <gazebo reference="right_wheel_link">
+    <laserRetro>${laser_retro}</laserRetro>
+  </gazebo>
+  <gazebo reference="caster_link">
+    <laserRetro>${laser_retro}</laserRetro>
   </gazebo>
   <gazebo reference="${imu_frame}">

File: src/gazebo_sim/robots/fishbot_v1/urdf/fishbot_v1.xacro (robot description, xacro)
@@ -20,4 +20,5 @@
   <xacro:property name="lidar_frame" value="${robot_cfg['lidar_frame']}"/>
   <xacro:property name="imu_frame" value="${robot_cfg['imu_frame']}"/>
+  <xacro:property name="laser_retro" value="${robot_cfg.get('laser_retro', 0.0)}"/>
   <xacro:property name="odom_frame" value="${robot_cfg['odom_frame']}"/>
   <xacro:property name="base_frame_prefixed" value="${frame_prefix + base_frame}"/>
@@ -214,7 +215,20 @@
       <publish_odom>${'true' if diff_drive_cfg['publish_odom'] else 'false'}</publish_odom>
       <publish_odom_tf>${'true' if diff_drive_cfg['publish_odom_tf'] else 'false'}</publish_odom_tf>
+      <tf_prefix>${frame_prefix}</tf_prefix>
       <odometry_frame>${odom_frame_prefixed}</odometry_frame>
       <robot_base_frame>${base_frame_prefixed}</robot_base_frame>
     </plugin>
+  </gazebo>
+  <gazebo reference="${base_frame}">
+    <laserRetro>${laser_retro}</laserRetro>
+  </gazebo>
+  <gazebo reference="left_wheel_link">
+    <laserRetro>${laser_retro}</laserRetro>
+  </gazebo>
+  <gazebo reference="right_wheel_link">
+    <laserRetro>${laser_retro}</laserRetro>
+  </gazebo>
+  <gazebo reference="caster_link">
+    <laserRetro>${laser_retro}</laserRetro>
   </gazebo>
   <gazebo reference="${imu_frame}">

File: src/gazebo_sim/robots/fishbot_v2_3d/urdf/fishbot_v2_3d.xacro (robot description, xacro)
@@ -21,4 +21,5 @@
   <xacro:property name="imu_frame" value="${robot_cfg['imu_frame']}"/>
   <xacro:property name="odom_frame" value="${robot_cfg['odom_frame']}"/>
+  <xacro:property name="laser_retro" value="${robot_cfg.get('laser_retro', 0.0)}"/>
   <xacro:property name="base_frame_prefixed" value="${frame_prefix + base_frame}"/>
   <xacro:property name="lidar_frame_prefixed" value="${frame_prefix + lidar_frame}"/>
@@ -214,7 +215,20 @@
       <publish_odom>${'true' if diff_drive_cfg['publish_odom'] else 'false'}</publish_odom>
       <publish_odom_tf>${'true' if diff_drive_cfg['publish_odom_tf'] else 'false'}</publish_odom_tf>
+      <tf_prefix>${frame_prefix}</tf_prefix>
       <odometry_frame>${odom_frame_prefixed}</odometry_frame>
       <robot_base_frame>${base_frame_prefixed}</robot_base_frame>
     </plugin>
+  </gazebo>
+  <gazebo reference="${base_frame}">
+    <laserRetro>${laser_retro}</laserRetro>
+  </gazebo>
+  <gazebo reference="left_wheel_link">
+    <laserRetro>${laser_retro}</laserRetro>
+  </gazebo>
+  <gazebo reference="right_wheel_link">
+    <laserRetro>${laser_retro}</laserRetro>
+  </gazebo>
+  <gazebo reference="caster_link">
+    <laserRetro>${laser_retro}</laserRetro>
   </gazebo>
   <gazebo reference="${imu_frame}">
