Commit message: fix frame names

File: src/gazebo_sim/robots/fishbot_v2_3d/urdf/fishbot_v2_3d.xacro (robot description, xacro)
@@ -3,59 +3,69 @@
   <xacro:arg name="config_file" default="$(find gazebo_sim)/robots/fishbot_v2_3d/config/fishbot_v2_3d.yaml"/>
   <xacro:arg name="robot_namespace" default=""/>
-  <xacro:property name="config_file" value="$(arg config_file)"/>
+  <!-- Load YAML config -->
   <xacro:property name="robot_namespace" value="$(arg robot_namespace)"/>
-  <xacro:property name="frame_prefix" value="${robot_namespace + '/' if robot_namespace != '' else ''}"/>
-  <xacro:property name="cfg" value="${xacro.load_yaml(config_file)}"/>
-  <xacro:property name="robot_cfg" value="${cfg['robot']}"/>
-  <xacro:property name="geometry_cfg" value="${cfg['geometry']}"/>
+  <xacro:property name="config_file"    value="$(arg config_file)"/>
+  <xacro:property name="cfg"            value="${xacro.load_yaml(config_file)}"/>
+  <xacro:property name="robot_cfg"      value="${cfg['robot']}"/>
+  <xacro:property name="geometry_cfg"   value="${cfg['geometry']}"/>
   <xacro:property name="kinematics_cfg" value="${cfg['kinematics']}"/>
-  <xacro:property name="plugins_cfg" value="${cfg['plugins']}"/>
-  <xacro:property name="imu_cfg" value="${cfg['imu']}"/>
-  <xacro:property name="lidar_cfg" value="${cfg['lidar']}"/>
-  <xacro:property name="base_geom" value="${geometry_cfg['base']}"/>
-  <xacro:property name="wheel_geom" value="${geometry_cfg['wheel']}"/>
+  <xacro:property name="plugins_cfg"    value="${cfg['plugins']}"/>
+  <xacro:property name="imu_cfg"        value="${cfg['imu']}"/>
+  <xacro:property name="lidar_cfg"      value="${cfg['lidar']}"/>
+  <!-- Namespacing -->
+  <xacro:property name="ns"           value="${robot_namespace}"/>
+  <xacro:property name="frame_prefix" value="${ns + '/' if ns != '' else ''}"/>
+  <xacro:property name="topic_prefix" value="${'/' + ns if ns != '' else ''}"/>
+  <!-- Frames -->
+  <xacro:property name="base_frame"  value="${robot_cfg['base_frame']}"/>
+  <xacro:property name="lidar_frame" value="${robot_cfg['lidar_frame']}"/>
+  <xacro:property name="imu_frame"   value="${robot_cfg['imu_frame']}"/>
+  <xacro:property name="odom_frame"  value="${robot_cfg['odom_frame']}"/>
+  <xacro:property name="base_frame_prefixed"  value="${frame_prefix + base_frame}"/>
+  <xacro:property name="lidar_frame_prefixed" value="${frame_prefix + lidar_frame}"/>
+  <xacro:property name="imu_frame_prefixed"   value="${frame_prefix + imu_frame}"/>
+  <xacro:property name="odom_frame_prefixed"  value="${frame_prefix + odom_frame}"/>
+  <!-- Topics -->
+  <xacro:property name="odom_topic"    value="${topic_prefix + '/' + robot_cfg['odom_pub']}"/>
+  <xacro:property name="lidar_topic"   value="${topic_prefix + '/' + robot_cfg['lidar_pub']}"/>
+  <xacro:property name="imu_topic"     value="${topic_prefix + '/' + robot_cfg['imu_pub']}"/>
+  <xacro:property name="cmd_vel_topic" value="${topic_prefix + '/cmd_vel'}"/>
+  <!-- Geometry config -->
+  <xacro:property name="base_geom"   value="${geometry_cfg['base']}"/>
+  <xacro:property name="wheel_geom"  value="${geometry_cfg['wheel']}"/>
   <xacro:property name="caster_geom" value="${geometry_cfg['caster']}"/>
-  <xacro:property name="diff_drive_cfg" value="${plugins_cfg['diff_drive']}"/>
-  <xacro:property name="base_frame" value="${robot_cfg['base_frame']}"/>
-  <xacro:property name="lidar_frame" value="${robot_cfg['lidar_frame']}"/>
-  <xacro:property name="imu_frame" value="${robot_cfg['imu_frame']}"/>
-  <xacro:property name="odom_frame" value="${robot_cfg['odom_frame']}"/>
-  <xacro:property name="laser_retro" value="${robot_cfg.get('laser_retro', 0.0)}"/>
-  <xacro:property name="base_frame_prefixed" value="${frame_prefix + base_frame}"/>
-  <xacro:property name="lidar_frame_prefixed" value="${frame_prefix + lidar_frame}"/>
-  <xacro:property name="imu_frame_prefixed" value="${frame_prefix + imu_frame}"/>
-  <xacro:property name="odom_frame_prefixed" value="${frame_prefix + odom_frame}"/>
-  <xacro:property name="odom_pub" value="${robot_cfg['odom_pub']}"/>
-  <xacro:property name="lidar_pub" value="${robot_cfg['lidar_pub']}"/>
-  <xacro:property name="imu_pub" value="${robot_cfg['imu_pub']}"/>
-  <xacro:property name="topic_prefix" value="${'/' + robot_namespace if robot_namespace else ''}"/>
-  <xacro:property name="odom_topic" value="${topic_prefix + '/' + odom_pub if topic_prefix else '/' + odom_pub}"/>
-  <xacro:property name="lidar_topic" value="${topic_prefix + '/' + lidar_pub if topic_prefix else '/' + lidar_pub}"/>
-  <xacro:property name="imu_topic" value="${topic_prefix + '/' + imu_pub if topic_prefix else '/' + imu_pub}"/>
-  <xacro:property name="cmd_vel_topic" value="${topic_prefix + '/cmd_vel' if topic_prefix else '/cmd_vel'}"/>
-  <xacro:property name="tf_topic" value="/tf"/>
-  <xacro:property name="wheel_radius" value="${wheel_geom['radius']}"/>
-  <xacro:property name="wheel_length" value="${wheel_geom['length']}"/>
+  <xacro:property name="wheel_radius"  value="${wheel_geom['radius']}"/>
+  <xacro:property name="wheel_length"  value="${wheel_geom['length']}"/>
   <xacro:property name="wheel_inertia" value="${wheel_geom['inertia_diag']}"/>
   <xacro:property name="caster_radius" value="${caster_geom['radius']}"/>
   <xacro:property name="base_radius" value="${base_geom['cyl_radius']}"/>
   <xacro:property name="base_length" value="${base_geom['cyl_length']}"/>
-  <xacro:property name="wheel_mass" value="${wheel_geom['mass']}"/>
-  <xacro:property name="base_mass" value="${base_geom['mass']}"/>
+  <xacro:property name="wheel_mass"  value="${wheel_geom['mass']}"/>
+  <xacro:property name="base_mass"   value="${base_geom['mass']}"/>
   <xacro:property name="caster_mass" value="${caster_geom['mass']}"/>
   <xacro:property name="base_ixx" value="${base_geom['inertia']['ixx']}"/>
   <xacro:property name="base_iyy" value="${base_geom['inertia']['iyy']}"/>
   <xacro:property name="base_izz" value="${base_geom['inertia']['izz']}"/>
-  <xacro:property name="wheel_sep" value="${kinematics_cfg['wheel_separation']}"/>
-  <xacro:property name="wheel_diameter" value="${kinematics_cfg['wheel_diameter']}"/>
-  <link name="base_footprint"/>
-  <joint name="base_joint" type="fixed">
-    <parent link="base_footprint"/>
-    <child link="${base_frame}"/>
-    <origin xyz="0.0 0.0 0.076" rpy="0 0 0"/>
-  </joint>
+  <!-- Kinematics / diff drive -->
+  <xacro:property name="kin_cfg"        value="${kinematics_cfg}"/>
+  <xacro:property name="wheel_sep"      value="${kin_cfg['wheel_separation']}"/>
+  <xacro:property name="wheel_diameter" value="${kin_cfg['wheel_diameter']}"/>
+  <xacro:property name="diff_drive_cfg"   value="${plugins_cfg['diff_drive']}"/>
+  <xacro:property name="diff_update_rate" value="${diff_drive_cfg['update_rate']}"/>
+  <!-- Laser retro from config -->
+  <xacro:property name="laser_retro" value="${robot_cfg.get('laser_retro', 0.0)}"/>
+  <!-- Height layout: wheels / caster on ground, base body above -->
+  <xacro:property name="base_clearance" value="0.01"/>
+  <xacro:property name="base_z_offset" value="${wheel_radius + base_clearance + base_length * 0.5}"/>
+  <xacro:property name="base_top_z"    value="${base_z_offset + base_length * 0.5}"/>
+  <xacro:property name="lidar_joint_z" value="${base_top_z + 0.02}"/>
+  <xacro:property name="imu_joint_z"   value="${base_z_offset}"/>
+  <!-- ========================================================= -->
+  <!-- GEOMETRY links + joints                                  -->
+  <!-- ========================================================= -->
+  <!-- Base link -->
   <link name="${base_frame}">
     <visual>
-      <origin xyz="0 0 0.0" rpy="0 0 0"/>
+      <origin xyz="0 0 ${base_z_offset}" rpy="0 0 0"/>
       <geometry>
         <cylinder length="${base_length}" radius="${base_radius}"/>
@@ -66,5 +76,5 @@
     </visual>
     <collision>
-      <origin xyz="0 0 0.0" rpy="0 0 0"/>
+      <origin xyz="0 0 ${base_z_offset}" rpy="0 0 0"/>
       <geometry>
         <cylinder length="${base_length}" radius="${base_radius}"/>
@@ -76,4 +86,5 @@
     </inertial>
   </link>
+  <!-- Lidar link -->
   <link name="${lidar_frame}">
     <visual>
@@ -100,6 +111,7 @@
     <parent link="${base_frame}"/>
     <child link="${lidar_frame}"/>
-    <origin xyz="0 0 0.075"/>
-  </joint>
+    <origin xyz="0 0 ${lidar_joint_z}" rpy="0 0 0"/>
+  </joint>
+  <!-- IMU link -->
   <link name="${imu_frame}">
     <visual>
@@ -123,6 +135,7 @@
     <parent link="${base_frame}"/>
     <child link="${imu_frame}"/>
-    <origin xyz="0 0 0.02"/>
-  </joint>
+    <origin xyz="0 0 ${imu_joint_z}" rpy="0 0 0"/>
+  </joint>
+  <!-- Wheels -->
   <link name="left_wheel_link">
     <visual>
@@ -161,8 +174,9 @@
     </inertial>
   </link>
+  <!-- Wheel centers at wheel_radius -> bottom at z = 0 -->
   <joint name="left_wheel_joint" type="continuous">
     <parent link="${base_frame}"/>
     <child link="left_wheel_link"/>
-    <origin xyz="-0.02 0.10 -0.06"/>
+    <origin xyz="-0.02 0.10 ${wheel_radius}" rpy="0 0 0"/>
     <axis xyz="0 1 0"/>
   </joint>
@@ -170,7 +184,8 @@
     <parent link="${base_frame}"/>
     <child link="right_wheel_link"/>
-    <origin xyz="-0.02 -0.10 -0.06"/>
+    <origin xyz="-0.02 -0.10 ${wheel_radius}" rpy="0 0 0"/>
     <axis xyz="0 1 0"/>
   </joint>
+  <!-- Caster -->
   <link name="caster_link">
     <visual>
@@ -191,10 +206,15 @@
     </inertial>
   </link>
+  <!-- Caster center at caster_radius -> bottom at z = 0 -->
   <joint name="caster_joint" type="fixed">
     <parent link="${base_frame}"/>
     <child link="caster_link"/>
-    <origin xyz="0.06 0.0 -0.076"/>
+    <origin xyz="0.06 0.0 ${caster_radius}" rpy="0 0 0"/>
     <axis xyz="0 1 0"/>
   </joint>
+  <!-- ========================================================= -->
+  <!-- GAZEBO PLUGINS / EXTRAS                                   -->
+  <!-- ========================================================= -->
+  <!-- Gazebo visuals / friction -->
   <gazebo reference="caster_link">
     <material>Gazebo/Black</material>
@@ -206,9 +226,10 @@
     <kd value="10.0"/>
   </gazebo>
+  <!-- Diff-drive plugin -->
   <gazebo>
     <plugin
         filename="ignition-gazebo-diff-drive-system"
         name="ignition::gazebo::systems::DiffDrive">
-      <odom_publish_frequency>${diff_drive_cfg['update_rate']}</odom_publish_frequency>
+      <odom_publish_frequency>${diff_update_rate}</odom_publish_frequency>
       <left_joint>left_wheel_joint</left_joint>
       <right_joint>right_wheel_joint</right_joint>
@@ -217,9 +238,10 @@
       <topic>${cmd_vel_topic}</topic>
       <odom_topic>${odom_topic}</odom_topic>
-      <tf_topic>${tf_topic}</tf_topic>
+      <tf_topic>/tf</tf_topic>
       <frame_id>${odom_frame_prefixed}</frame_id>
       <child_frame_id>${base_frame_prefixed}</child_frame_id>
     </plugin>
   </gazebo>
+  <!-- Laser retro -->
   <gazebo reference="${base_frame}">
     <laserRetro>${laser_retro}</laserRetro>
@@ -234,4 +256,8 @@
     <laserRetro>${laser_retro}</laserRetro>
   </gazebo>
+  <!-- ========================================================= -->
+  <!-- SENSORS (Gazebo sensors attached to links)                -->
+  <!-- ========================================================= -->
+  <!-- IMU sensor -->
   <gazebo reference="${imu_frame}">
     <sensor name="imu_sensor" type="imu">
@@ -240,5 +266,5 @@
       <visualize>${'true' if imu_cfg['visualize'] else 'false'}</visualize>
       <topic>${imu_topic}</topic>
-      <frame_id>${imu_frame_prefixed}</frame_id>
+      <gz_frame_id>${imu_frame_prefixed}</gz_frame_id>
       <enable_metrics>true</enable_metrics>
       <imu>
@@ -298,4 +324,5 @@
     </sensor>
   </gazebo>
+  <!-- Lidar sensor -->
   <gazebo reference="${lidar_frame}">
     <sensor name="lidar_sensor" type="gpu_lidar">
@@ -303,7 +330,6 @@
       <visualize>${'true' if lidar_cfg['visualize'] else 'false'}</visualize>
       <update_rate>${lidar_cfg['update_rate']}</update_rate>
-      <pose>0 0 0.075 0 0 0</pose>
       <topic>${lidar_topic}</topic>
-      <frame_id>${lidar_frame_prefixed}</frame_id>
+      <gz_frame_id>${lidar_frame_prefixed}</gz_frame_id>
       <lidar>
         <scan>

Commit message: fix: lidar intensity

File: src/gazebo_sim/robots/fishbot_mid360/urdf/fishbot_mid360.xacro (robot description, xacro)
@@ -243,16 +243,19 @@
     </plugin>
   </gazebo>
-  <!-- Laser retro -->
+  <!-- High LiDAR reflectivity on robot body -->
   <gazebo reference="${base_frame}">
-    <laserRetro>${laser_retro}</laserRetro>
+    <visual><laser_retro>${laser_retro}</laser_retro></visual>
+  </gazebo>
+  <gazebo reference="${lidar_frame}">
+    <visual><laser_retro>${laser_retro}</laser_retro></visual>
   </gazebo>
   <gazebo reference="left_wheel_link">
-    <laserRetro>${laser_retro}</laserRetro>
+    <visual><laser_retro>${laser_retro}</laser_retro></visual>
   </gazebo>
   <gazebo reference="right_wheel_link">
-    <laserRetro>${laser_retro}</laserRetro>
+    <visual><laser_retro>${laser_retro}</laser_retro></visual>
   </gazebo>
   <gazebo reference="caster_link">
-    <laserRetro>${laser_retro}</laserRetro>
+    <visual><laser_retro>${laser_retro}</laser_retro></visual>
   </gazebo>
   <!-- ========================================================= -->

File: src/gazebo_sim/robots/fishbot_v1/urdf/fishbot_v1.xacro (robot description, xacro)
@@ -243,16 +243,19 @@
     </plugin>
   </gazebo>
-  <!-- Laser retro -->
+  <!-- High LiDAR reflectivity on robot body -->
   <gazebo reference="${base_frame}">
-    <laserRetro>${laser_retro}</laserRetro>
+    <visual><laser_retro>${laser_retro}</laser_retro></visual>
+  </gazebo>
+  <gazebo reference="${lidar_frame}">
+    <visual><laser_retro>${laser_retro}</laser_retro></visual>
   </gazebo>
   <gazebo reference="left_wheel_link">
-    <laserRetro>${laser_retro}</laserRetro>
+    <visual><laser_retro>${laser_retro}</laser_retro></visual>
   </gazebo>
   <gazebo reference="right_wheel_link">
-    <laserRetro>${laser_retro}</laserRetro>
+    <visual><laser_retro>${laser_retro}</laser_retro></visual>
   </gazebo>
   <gazebo reference="caster_link">
-    <laserRetro>${laser_retro}</laserRetro>
+    <visual><laser_retro>${laser_retro}</laser_retro></visual>
   </gazebo>
   <!-- ========================================================= -->

File: src/gazebo_sim/robots/fishbot_v2_3d/urdf/fishbot_v2_3d.xacro (robot description, xacro)
@@ -243,16 +243,19 @@
     </plugin>
   </gazebo>
-  <!-- Laser retro -->
+  <!-- High LiDAR reflectivity on robot body -->
   <gazebo reference="${base_frame}">
-    <laserRetro>${laser_retro}</laserRetro>
+    <visual><laser_retro>${laser_retro}</laser_retro></visual>
+  </gazebo>
+  <gazebo reference="${lidar_frame}">
+    <visual><laser_retro>${laser_retro}</laser_retro></visual>
   </gazebo>
   <gazebo reference="left_wheel_link">
-    <laserRetro>${laser_retro}</laserRetro>
+    <visual><laser_retro>${laser_retro}</laser_retro></visual>
   </gazebo>
   <gazebo reference="right_wheel_link">
-    <laserRetro>${laser_retro}</laserRetro>
+    <visual><laser_retro>${laser_retro}</laser_retro></visual>
   </gazebo>
   <gazebo reference="caster_link">
-    <laserRetro>${laser_retro}</laserRetro>
+    <visual><laser_retro>${laser_retro}</laser_retro></visual>
   </gazebo>
   <!-- ========================================================= -->

Commit message: fix: support to disable odom

File: src/gazebo_sim/robots/fishbot_mid360/urdf/fishbot_mid360.xacro (robot description, xacro)
@@ -53,4 +53,9 @@
   <xacro:property name="diff_drive_cfg"   value="${plugins_cfg['diff_drive']}"/>
   <xacro:property name="diff_update_rate" value="${diff_drive_cfg['update_rate']}"/>
+  <xacro:property name="diff_publish_odom_bool" value="${bool(diff_drive_cfg.get('publish_odom', True))}"/>
+  <xacro:property name="diff_publish_tf_bool"   value="${bool(diff_drive_cfg.get('publish_odom_tf', True))}"/>
+  <xacro:property name="diff_publish_odom" value="${'true' if diff_publish_odom_bool else 'false'}"/>
+  <xacro:property name="diff_publish_tf"   value="${'true' if diff_publish_tf_bool else 'false'}"/>
+  <xacro:property name="diff_tf_topic"     value="${'/tf' if diff_publish_tf_bool else '/tf_disabled'}"/>
   <!-- Laser retro from config -->
   <xacro:property name="laser_retro" value="${robot_cfg.get('laser_retro', 0.0)}"/>
@@ -238,7 +243,9 @@
       <topic>${cmd_vel_topic}</topic>
       <odom_topic>${odom_topic}</odom_topic>
-      <tf_topic>/tf</tf_topic>
-      <frame_id>${odom_frame_prefixed}</frame_id>
-      <child_frame_id>${base_frame_prefixed}</child_frame_id>
+      <tf_topic>${diff_tf_topic}</tf_topic>
+      <odom_frame>${odom_frame_prefixed}</odom_frame>
+      <robot_base_frame>${base_frame_prefixed}</robot_base_frame>
+      <publish_odom>${diff_publish_odom}</publish_odom>
+      <publish_tf>${diff_publish_tf}</publish_tf>
     </plugin>
   </gazebo>

File: src/gazebo_sim/robots/fishbot_v1/urdf/fishbot_v1.xacro (robot description, xacro)
@@ -53,4 +53,9 @@
   <xacro:property name="diff_drive_cfg"   value="${plugins_cfg['diff_drive']}"/>
   <xacro:property name="diff_update_rate" value="${diff_drive_cfg['update_rate']}"/>
+  <xacro:property name="diff_publish_odom_bool" value="${bool(diff_drive_cfg.get('publish_odom', True))}"/>
+  <xacro:property name="diff_publish_tf_bool"   value="${bool(diff_drive_cfg.get('publish_odom_tf', True))}"/>
+  <xacro:property name="diff_publish_odom" value="${'true' if diff_publish_odom_bool else 'false'}"/>
+  <xacro:property name="diff_publish_tf"   value="${'true' if diff_publish_tf_bool else 'false'}"/>
+  <xacro:property name="diff_tf_topic"     value="${'/tf' if diff_publish_tf_bool else '/tf_disabled'}"/>
   <!-- Laser retro from config -->
   <xacro:property name="laser_retro" value="${robot_cfg.get('laser_retro', 0.0)}"/>
@@ -238,7 +243,9 @@
       <topic>${cmd_vel_topic}</topic>
       <odom_topic>${odom_topic}</odom_topic>
-      <tf_topic>/tf</tf_topic>
-      <frame_id>${odom_frame_prefixed}</frame_id>
-      <child_frame_id>${base_frame_prefixed}</child_frame_id>
+      <tf_topic>${diff_tf_topic}</tf_topic>
+      <odom_frame>${odom_frame_prefixed}</odom_frame>
+      <robot_base_frame>${base_frame_prefixed}</robot_base_frame>
+      <publish_odom>${diff_publish_odom}</publish_odom>
+      <publish_tf>${diff_publish_tf}</publish_tf>
     </plugin>
   </gazebo>

File: src/gazebo_sim/robots/fishbot_v2_3d/urdf/fishbot_v2_3d.xacro (robot description, xacro)
@@ -53,4 +53,9 @@
   <xacro:property name="diff_drive_cfg"   value="${plugins_cfg['diff_drive']}"/>
   <xacro:property name="diff_update_rate" value="${diff_drive_cfg['update_rate']}"/>
+  <xacro:property name="diff_publish_odom_bool" value="${bool(diff_drive_cfg.get('publish_odom', True))}"/>
+  <xacro:property name="diff_publish_tf_bool"   value="${bool(diff_drive_cfg.get('publish_odom_tf', True))}"/>
+  <xacro:property name="diff_publish_odom" value="${'true' if diff_publish_odom_bool else 'false'}"/>
+  <xacro:property name="diff_publish_tf"   value="${'true' if diff_publish_tf_bool else 'false'}"/>
+  <xacro:property name="diff_tf_topic"     value="${'/tf' if diff_publish_tf_bool else '/tf_disabled'}"/>
   <!-- Laser retro from config -->
   <xacro:property name="laser_retro" value="${robot_cfg.get('laser_retro', 0.0)}"/>
@@ -277,7 +282,9 @@
       <topic>${cmd_vel_topic}</topic>
       <odom_topic>${odom_topic}</odom_topic>
-      <tf_topic>/tf</tf_topic>
-      <frame_id>${odom_frame_prefixed}</frame_id>
-      <child_frame_id>${base_frame_prefixed}/wheel</child_frame_id>
+      <tf_topic>${diff_tf_topic}</tf_topic>
+      <odom_frame>${odom_frame_prefixed}</odom_frame>
+      <robot_base_frame>${base_frame_prefixed}</robot_base_frame>
+      <publish_odom>${diff_publish_odom}</publish_odom>
+      <publish_tf>${diff_publish_tf}</publish_tf>
     </plugin>
   </gazebo>
